File: HW/Node/with_solar.sch (EAGLE design)
At the start: 27 parts, among them U1 MS560702BA03-50, U2 HDC2080DMBR, U3 RFM69HW, U4 LTC3106, X1 734120110

Commit message: HW: Update node schematic and board
Signed-off-by: Ales Musil <aedvin1@gmail.com>
Connections:
- new net RFM_INT: STM32L031K6_1.PA1, U3.DIO0
Changed lines of the file:
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@@
 <setting verticaltext="up"/>
 </settings>
-<grid distance="0.1" unitdist="inch" unit="inch" style="lines" multiple="1" display="no" altdistance="0.01" altunitdist="inch" altunit="inch"/>
+<grid distance="0.05" unitdist="inch" unit="inch" style="lines" multiple="1" display="no" altdistance="0.01" altunitdist="inch" altunit="inch"/>
 <layers>
 <layer number="1" name="Top" color="4" fill="1" visible="no" active="no"/>
@@
 </segment>
 </net>
+<net name="RFM_INT" class="0">
+<segment>
+<pinref part="STM32L031K6_1" gate="G$1" pin="PA1"/>
+<wire x1="38.1" y1="68.58" x2="31.75" y2="68.58" width="0.1524" layer="91"/>
+<label x="26.67" y="68.58" size="1.778" layer="95"/>
+</segment>
+<segment>
+<pinref part="U3" gate="G$1" pin="DIO0"/>
+<wire x1="96.52" y1="5.08" x2="102.87" y2="5.08" width="0.1524" layer="91"/>
+<label x="96.52" y="5.08" size="1.778" layer="95"/>
+</segment>
+</net>
